File: TurnTimer.kicad_pcb (KiCad board)
At the start: 2 copper layers, 100 x 100 mm, 22 parts, among them SW1 SW_Push, SW2 SW_Push, SW3 SW_Push, SW4 SW_Push, SW5 SW_Push, SW6 SW_Push, SW7 SW_Push, SW8 SW_Push

Commit message: absorbed 096 into one repo
Parts:
- removed BatterBarrelJack1: Barrel_Jack_Switch, Connector_BarrelJack:BarrelJack_CUI_PJ-102AH_Horizontal
- removed REF**: MountingHole_3.2mm_M3, MountingHole:MountingHole_3.2mm_M3
- added H1: MountingHole, MountingHole:MountingHole_3.2mm_M3, F.Cu at (143.4, 98.7)
- added J1: Screw_Terminal_01x02, TerminalBlock_CUI:TerminalBlock_CUI_TB007-508-02_1x02_P5.08mm_Horizontal, F.Cu at (106.5, 71.5)
- moved PanelSwitchConn1 13.7 mm to (107.2, 85.0), turned to 90 degrees
Connections:
- PanelSwitchConn1 pad 1: /PWR_IN -> /Battery9V+
Routing:
- net /Battery9V+: track 0.00 -> 13.8 mm
- net /PWR_IN: track 13.5 -> 0.00 mm
- net /V_IN: track 9.16 -> 15.7 mm
Other:
- board text added: "NEG-"
- board text added: "POS+"
- board text added: "R1"
