File: TurnTimer.kicad_sch (KiCad schematic)
At the start: 21 parts, among them SW1 SW_Push, SW2 SW_Push, SW3 SW_Push, SW4 SW_Push, SW5 SW_Push, SW6 SW_Push, SW7 SW_Push, SW8 SW_Push

Commit message: absorbed 096 into one repo
Parts:
- removed BatterBarrelJack1: Barrel_Jack_Switch, Connector_BarrelJack:BarrelJack_CUI_PJ-102AH_Horizontal, symbol Connector:Barrel_Jack_Switch
- added H1: MountingHole, MountingHole:MountingHole_3.2mm_M3, symbol Mechanical:MountingHole
- added J1: Screw_Terminal_01x02, TerminalBlock_CUI:TerminalBlock_CUI_TB007-508-02_1x02_P5.08mm_Horizontal, symbol Connector:Screw_Terminal_01x02
Connections:
- net GND: now also J1.2 (Pin_2)
- net PWR_IN renamed Battery9V+
- net Battery9V+: now also J1.1 (Pin_1)
- no-connect marks 16 -> 15
Other:
- moved on the sheet: PanelSwitchConn1
